Commit message: Day17: spawn custom robot in Gazebo with lidar visualization

File: workspace/src/my_robot_description/urdf/my_robot.urdf (robot description, URDF)
Before this commit: robot my_robot, 6 links, 5 joints
Joints:
- joint base_joint: origin xyz=0 0 0.1 rpy=0 0 0 -> xyz=0 0 0.15 rpy=0 0 0
- joint caster_wheel_joint: origin xyz=0.2 0 -0.05 rpy=0 0 0 -> xyz=0.2 0 -0.07 rpy=0 0 0
- joint left_wheel_joint: origin xyz=0 0.225 0 rpy=-1.5708 0 0 -> xyz=0 0.225 -0.02 rpy=-1.5708 0 0
- joint right_wheel_joint: axis 0 0 1 -> 0 0 -1; origin xyz=0 -0.225 0 rpy=1.5708 0 0 -> xyz=0 -0.225 -0.02 rpy=1.5708 0 0

Commit message: Update URDF: add front marker sphere

File: workspace/src/my_robot_description/urdf/my_robot.urdf (robot description, URDF)
Before this commit: robot my_robot, 6 links, 5 joints
Links:
- link base_link: geometry collision box size=0.6 0.4 0.2; visual box size=0.6 0.4 0.2

Commit message: Day20: Nav2 tuning + URDF stability debugging

File: workspace/src/my_robot_description/urdf/my_robot.urdf (robot description, URDF)
Before this commit: robot my_robot, 6 links, 5 joints
Links:
- link base_link: geometry collision box size=0.6 0.4 0.2; visual box size=0.08 0.04 0.04
- link caster_wheel: mass 0.1 -> 0.05; geometry collision sphere radius=0.04; visual sphere radius=0.04
Joints:
- joint base_joint: origin xyz=0 0 0.15 rpy=0 0 0 -> xyz=0 0 0.16 rpy=0 0 0
- joint caster_wheel_joint: origin xyz=0.2 0 -0.07 rpy=0 0 0 -> xyz=-0.25 0 -0.06 rpy=0 0 0

Commit message: Day21: add rear support wheel to improve stability and refine URDF structure

File: workspace/src/my_robot_description/urdf/my_robot.urdf (robot description, URDF)
Before this commit: robot my_robot, 6 links, 5 joints
Links:
- removed link caster_wheel
- added link rear_support_wheel, mass 0.05; collision cylinder length=0.02 radius=0.03; visual cylinder length=0.02 radius=0.03
- link base_link: mass 5.0 -> 2.0; geometry collision box size=0.36 0.26 0.08; visual box size=0.05 0.04 0.03
- link left_wheel: mass 0.5 -> 0.25; geometry collision cylinder length=0.04 radius=0.08; visual cylinder length=0.04 radius=0.08
- link lidar_link: mass 0.1 -> 0.10
- link right_wheel: mass 0.5 -> 0.25; geometry collision cylinder length=0.04 radius=0.08; visual cylinder length=0.04 radius=0.08
Joints:
- removed joint caster_wheel_joint
- added joint rear_support_wheel_joint: type continuous, parent base_link, child rear_support_wheel, origin xyz=-0.14 0 -0.07 rpy=0 0 0, axis 0 1 0
- joint base_joint: origin xyz=0 0 0.16 rpy=0 0 0 -> xyz=0 0 0.14 rpy=0 0 0
- joint left_wheel_joint: axis 0 0 1 -> 0 1 0; origin xyz=0 0.225 -0.02 rpy=-1.5708 0 0 -> xyz=0 0.15 -0.06 rpy=0 0 0
- joint lidar_joint: origin xyz=0 0 0.12 rpy=0 0 0 -> xyz=0 0 0.07 rpy=0 0 0
- joint right_wheel_joint: axis 0 0 -1 -> 0 1 0; origin xyz=0 -0.225 -0.02 rpy=1.5708 0 0 -> xyz=0 -0.15 -0.06 rpy=0 0 0

Commit message: Day22: system stabilized, navigation closed-loop

File: workspace/src/my_robot_description/urdf/my_robot.urdf (robot description, URDF)
Before this commit: robot my_robot, 6 links, 5 joints
Links:
- link rear_support_wheel: mass 0.05 -> 0.08; geometry collision sphere radius=0.03; visual sphere radius=0.03
Joints:
- joint left_wheel_joint: origin xyz=0 0.15 -0.06 rpy=0 0 0 -> xyz=0.03 0.15 -0.06 rpy=0 0 0
- joint rear_support_wheel_joint: axis 0 1 0 -> (none); origin xyz=-0.14 0 -0.07 rpy=0 0 0 -> xyz=-0.12 0 -0.11 rpy=0 0 0; type continuous -> fixed
- joint right_wheel_joint: origin xyz=0 -0.15 -0.06 rpy=0 0 0 -> xyz=0.03 -0.15 -0.06 rpy=0 0 0
